Commit message: Update chassis.xacro

File: yegna_robot/src/yegna_pkg/src/chassis.xacro (robot description, xacro)
@@ -2,5 +2,5 @@
 <robot name="simple_legged_robot" xmlns:xacro="http://ros.org/wiki/xacro">
   <!-- Macro for simple_legged_robot body.  -->
-  	<xacro:include filename="chassis.gazebo" />
+  <xacro:include filename="chassis.gazebo" />
    <link name = "base_link"/>
    <joint name="base_link_to_body_joint" type="fixed">
@@ -8,5 +8,5 @@
       <child link="body_link"/>
     </joint>
-  	<link name="body_link">
+  <link name="body_link">
     <inertial>
       <origin xyz="-0.003053 -0.038651 -0.019268" />
@@ -31,5 +31,5 @@
     </collision>
   </link>
-  	<link name="camera_head">
+   <link name="camera_head">
     <inertial>
       <origin xyz="0.000064 -0.018565 -0.007667" />
@@ -131,5 +131,5 @@
     </collision>
   </link>
-	  <joint name="body_back_left_joint" type="fixed">
+ 	  <joint name="body_back_left_joint" type="fixed">
         <parent link="body_link"/>
           <child link="body_back_left"/>
@@ -143,5 +143,4 @@
                 </geometry>
                <!-- <origin xyz="0 0 -0.3" rpy="0 1.57075 0" /> -->
-              <!-- <origin xyz="-0.13522619 -0.010264050 0.0013935747" /> -->
                <origin xyz="-0.05 -0.010264050 0.0013935747" />
 	    	<material name="Blue">
@@ -309,6 +308,5 @@
                 </geometry>
                <!-- <origin xyz="0 0 -0.3" rpy="0 1.57075 0" /> -->
-               <!--  <origin xyz="0.13523 -0.010264 0.001394" /> -->
-                <origin xyz="0.05 -0.010264 0.001394"/>
+              <origin xyz="0.05 -0.010264 0.001394"/>
 	    	<material name="Blue">
 	    	  <color rgba = "0.0 0.0 0.80 1.0"/>
